Commit message: relative path to model fixed

File: roboracer_ws/src/roboracer_description/urdf/f1tenth_chassis.urdf (robot description, URDF)
Before this commit: robot roboracer_robot, 11 links, 10 joints
Links:
- link car_1_chassis: geometry collision box size=0.5 0.3 0.1; visual mesh filename=package://roboracer_description/meshes/chassis.stl scale=0.000990 0.0009375 0.0009375
- link car_1_laser: geometry collision box size=0.01 0.01 0.01; visual mesh filename=package://roboracer_description/meshes/laser_link.STL
- link car_1_left_front_wheel: geometry collision cylinder length=0.045 radius=0.05; visual mesh filename=package://roboracer_description/meshes/left_wheel.stl
- link car_1_left_rear_wheel: geometry collision cylinder length=0.045 radius=0.05; visual mesh filename=package://roboracer_description/meshes/left_wheel.stl
- link car_1_left_steering_hinge: geometry visual mesh filename=package://roboracer_description/meshes/hinge.stl
- link car_1_right_front_wheel: geometry collision cylinder length=0.045 radius=0.05; visual mesh filename=package://roboracer_description/meshes/right_wheel.stl
- link car_1_right_rear_wheel: geometry collision cylinder length=0.045 radius=0.05; visual mesh filename=package://roboracer_description/meshes/right_wheel.stl
- link car_1_right_steering_hinge: geometry visual mesh filename=package://roboracer_description/meshes/hinge.stl

Commit message: left wall bug updated

File: roboracer_ws/src/roboracer_description/urdf/f1tenth_chassis.urdf (robot description, URDF)
Before this commit: robot roboracer_robot, 11 links, 10 joints
Links:
- link car_1_laser: geometry collision box size=0.01 0.01 0.01; visual mesh filename=package://roboracer_description/meshes/laser_link.stl
