Commit message: Work on Visual Odometry
1) Work on Visual Odometry
2) Yolo Detection
3) Work on ORB-SLAM3

File: src/install/roboracer_description/share/roboracer_description/urdf/f1tenth_chassis.urdf (robot description, URDF)
Before this commit: robot roboracer_robot, 11 links, 10 joints
Links:
- link car_1_laser: mass 0.073 -> 0.5
Joints:
- joint car_1_camera_joint: origin xyz=0.40 0 0.10 rpy=0 0 0 -> xyz=0.40 0 0.15 rpy=0 0 0; parent car_1_chassis -> car_1_base_link

File: src/roboracer_description/urdf/f1tenth_chassis.urdf (robot description, URDF)
Before this commit: robot roboracer_robot, 11 links, 10 joints
Joints:
- joint car_1_camera_joint: origin xyz=0.40 0 0.10 rpy=0 0 0 -> xyz=0.40 0 0.15 rpy=0 0 0; parent car_1_chassis -> car_1_base_link
