Commit message: Visual Odometry
1) Work on Visual Odometry
2) Change the parameter match with ORB-SLAM
3) Continue work on crash fixes

File: src/roboracer_description/urdf/f1tenth_chassis.urdf (robot description, URDF)
Before this commit: robot roboracer_robot, 11 links, 10 joints
Joints:
- joint imu_joint: parent car_1_chassis -> car_1_base_link
